Commit message: Capture earlier uncommitted stack scripts, launch files and config
Not from today's session - this is pre-existing work that had never been
committed, added so the tree is clean and so today's commits reference files
that actually exist in history (start_navigation.sh, rviz_remote.launch.py and
others were untracked until now).

Includes the amr-stack systemd unit and supervisor, the start/stop scripts for
the full stack and mapping, the discovery-server scripts that were tried and
reverted on 2026-10-07, the mapping/navigation launch files, twist_mux and
mapper params, and the robot description edits.

Left out deliberately: "config/nav2_params (copy).yaml", a stale backup 175
diff lines adrift from the real file.

Co-Authored-By: Claude Opus 5 <noreply@anthropic.com>

File: description/lidar.xacro (robot description, xacro)
@@ -3,5 +3,5 @@
     <joint name="laser_joint" type="fixed">
     <parent link="chassis"/>  <child link="laser_frame"/>
-    <origin xyz="0.300 0 0.180" rpy="0 0 3.14159"/>
+    <origin xyz="0.310 0 0.180" rpy="0 0 0"/>
     </joint>
     <link name="laser_frame">

File: description/robot_core.xacro (robot description, xacro)
@@ -3,7 +3,7 @@
     <xacro:include filename="inertial_macros.xacro" />
     <!-- ===== dims (m) ===== -->
-    <xacro:property name="chassis_length" value="0.797"/>
-    <xacro:property name="chassis_width"  value="0.498"/>
-    <xacro:property name="chassis_height" value="0.170"/>
+    <xacro:property name="chassis_length" value="0.780"/>
+    <xacro:property name="chassis_width"  value="0.480"/>
+    <xacro:property name="chassis_height" value="0.180"/>
     <xacro:property name="chassis_mass"   value="10.0"/>
     <xacro:property name="wheel_radius" value="0.085"/>
